Commit message: Todo funcional faltante odometria

File: robot_bombero_description/urdf/arm.xacro (robot description, xacro)
@@ -116,5 +116,5 @@
     <parent link="link_waist"/>
     <child link="link_shoulder"/>
-    <origin xyz="0 0 ${height_waist}" rpy="0 0 0"/>
+    <origin xyz="0 0 ${height_waist}" rpy="0 -1.5708 0"/>
     <axis xyz="0 1 0"/>
     <limit effort="100" velocity="1.0" lower="-1.5" upper="1.5"/>
@@ -123,5 +123,5 @@
     <parent link="link_shoulder"/>
     <child link="link_elbow"/>
-    <origin xyz="0 0 ${height_shoulder}" rpy="0 0 0"/>
+    <origin xyz="0 0 ${height_shoulder}" rpy="0 -1.5708 0"/>
     <axis xyz="0 1 0"/>
     <limit effort="100" velocity="1.0" lower="-1.5" upper="1.5"/>
@@ -130,5 +130,5 @@
     <parent link="link_elbow"/>
     <child link="link_wrist"/>
-    <origin xyz="0 0 ${height_elbow}" rpy="0 0 0"/>
+    <origin xyz="0 0 ${height_elbow}" rpy="0 -1.5708 0"/>
     <axis xyz="0 1 0"/>
     <limit effort="100" velocity="1.0" lower="-1.5" upper="1.5"/>

File: robot_bombero_description/urdf/pump.xacro (robot description, xacro)
@@ -11,8 +11,9 @@
   </visual>
 </link>
-<joint name="joint_water_pump" type="fixed">
+<joint name="joint_water_pump" type="continuous">
   <parent link="chassis"/>
   <child link="water_pump_link"/>
   <origin xyz="-0.1 0 0.1" rpy="0 1.57 1.57"/>
+  <limit effort="100" velocity="1.0"/>
 </joint>
 </robot>

File: robot_bombero_description/urdf/robot.urdf.xacro (robot description, xacro)
@@ -10,4 +10,6 @@
   <xacro:robot_camera parent="link_wrist"/>
   <xacro:include filename="pump.xacro"/>
+  <!-- <xacro:include filename="transmissions.xacro"/>
+  <xacro:mecanum_transmissions/> -->
   <xacro:include filename="ros2_control.xacro"/>
   <xacro:robot_ros2_control/>

File: robot_bombero_description/urdf/ros2_control.xacro (robot description, xacro)
@@ -4,5 +4,5 @@
     <ros2_control name="FirebotSystem" type="system">
       <hardware>
-         <plugin>robot_bombero_hardware/FirebotHardwareInterface</plugin>
+         <plugin>robot_bombero_hardware/FireBotHardwareInterface</plugin>
           <param name="port_name">/dev/ttyUSB0</param>
       </hardware>
@@ -11,16 +11,20 @@
         <command_interface name="velocity"/>
         <state_interface name="velocity"/>
+        <state_interface name="position"/>
       </joint>
       <joint name="link_fr_wheel_joint">
         <command_interface name="velocity"/>
         <state_interface name="velocity"/>
+        <state_interface name="position"/>
       </joint>
       <joint name="link_rl_wheel_joint">
         <command_interface name="velocity"/>
         <state_interface name="velocity"/>
+        <state_interface name="position"/>
       </joint>
       <joint name="link_rr_wheel_joint">
         <command_interface name="velocity"/>
         <state_interface name="velocity"/>
+        <state_interface name="position"/>
       </joint>
       <!-- Articulaciones del brazo -->
@@ -45,5 +49,24 @@
         <command_interface name="effort"/>
         <state_interface name="effort"/>
+        <state_interface name="position"/>
       </joint>
+      <!--Informacion sensores -->
+      <sensor name="imu_sensor">
+        <state_interface name="angular_velocity.x"/>
+        <state_interface name="angular_velocity.y"/>
+        <state_interface name="angular_velocity.z"/>
+        <state_interface name="linear_acceleration.x"/>
+        <state_interface name="linear_acceleration.y"/>
+        <state_interface name="linear_acceleration.z"/>
+      </sensor>
+      <gpio name="sharp_front">
+        <state_interface name="analog_input"/>
+      </gpio>
+      <gpio name="sharp_left">
+        <state_interface name="analog_input"/>
+      </gpio>
+      <gpio name="sharp_right">
+        <state_interface name="analog_input"/>
+      </gpio>
     </ros2_control>
   </xacro:macro>

File: robot_bombero_description/urdf/sensors.xacro (robot description, xacro)
@@ -113,60 +113,4 @@
       <origin xyz="0 0 0.1" rpy="0 0 0"/>
     </joint>
-      <!-- Transmisiones para sensores IR -->
-    <transmission name="trans_ir_left">
-      <type>transmission_interface/SimpleTransmission</type>
-      <joint name="joint_sharp_left">
-        <hardwareInterface>hardware_interface/StateInterface</hardwareInterface>
-      </joint>
-      <actuator name="actuator_ir_left">
-        <hardwareInterface>hardware_interface/StateInterface</hardwareInterface>
-      </actuator>
-    </transmission>
-    <transmission name="trans_ir_center">
-      <type>transmission_interface/SimpleTransmission</type>
-      <joint name="joint_sharp_front">
-        <hardwareInterface>hardware_interface/StateInterface</hardwareInterface>
-      </joint>
-      <actuator name="actuator_ir_center">
-        <hardwareInterface>hardware_interface/StateInterface</hardwareInterface>
-      </actuator>
-    </transmission>
-    <transmission name="trans_ir_right">
-      <type>transmission_interface/SimpleTransmission</type>
-      <joint name="joint_sharp_right">
-        <hardwareInterface>hardware_interface/StateInterface</hardwareInterface>
-      </joint>
-      <actuator name="actuator_ir_right">
-        <hardwareInterface>hardware_interface/StateInterface</hardwareInterface>
-      </actuator>
-    </transmission>
-    <!-- Transmisiones para IMU -->
-    <transmission name="trans_imu_x">
-      <type>transmission_interface/SimpleTransmission</type>
-      <joint name="joint_imu">
-        <hardwareInterface>hardware_interface/StateInterface</hardwareInterface>
-      </joint>
-      <actuator name="actuator_imu_x">
-        <hardwareInterface>hardware_interface/StateInterface</hardwareInterface>
-      </actuator>
-    </transmission>
-    <transmission name="trans_imu_y">
-      <type>transmission_interface/SimpleTransmission</type>
-      <joint name="joint_imu">
-        <hardwareInterface>hardware_interface/StateInterface</hardwareInterface>
-      </joint>
-      <actuator name="actuator_imu_y">
-        <hardwareInterface>hardware_interface/StateInterface</hardwareInterface>
-      </actuator>
-    </transmission>
-    <transmission name="trans_imu_z">
-      <type>transmission_interface/SimpleTransmission</type>
-      <joint name="joint_imu">
-        <hardwareInterface>hardware_interface/StateInterface</hardwareInterface>
-      </joint>
-      <actuator name="actuator_imu_z">
-        <hardwareInterface>hardware_interface/StateInterface</hardwareInterface>
-      </actuator>
-    </transmission>
   </xacro:macro>
 </robot>

File: robot_bombero_description/urdf/wheels.xacro (robot description, xacro)
@@ -33,10 +33,10 @@
       <origin xyz="${xyz}" rpy="${rpy}"/>
       <axis xyz="0 0 1"/>
-      <limit effort="100" velocity="1.0" lower="0" upper="3.14"/>
+      <limit effort="100" velocity="1.0"/>
     </joint>
   </xacro:macro>
-  <xacro:mecanum_wheel name="link_fl_wheel" parent="base_link" xyz="0.25 0.17 0.05" rpy="1.5708 0 0"/>
-  <xacro:mecanum_wheel name="link_fr_wheel" parent="base_link" xyz="0.25 -0.17 0.05" rpy="1.5708 0 0"/>
-  <xacro:mecanum_wheel name="link_rl_wheel" parent="base_link" xyz="-0.25 0.17 0.05" rpy="1.5708 0 0"/>
-  <xacro:mecanum_wheel name="link_rr_wheel" parent="base_link" xyz="-0.25 -0.17 0.05" rpy="1.5708 0 0"/>
+  <xacro:mecanum_wheel name="link_fl_wheel" parent="base_link" xyz="0.25 0.17 0.05" rpy="-1.5708 0 0"/>
+  <xacro:mecanum_wheel name="link_fr_wheel" parent="base_link" xyz="0.25 -0.17 0.05" rpy="-1.5708 0 0"/>
+  <xacro:mecanum_wheel name="link_rl_wheel" parent="base_link" xyz="-0.25 0.17 0.05" rpy="-1.5708 0 0"/>
+  <xacro:mecanum_wheel name="link_rr_wheel" parent="base_link" xyz="-0.25 -0.17 0.05" rpy="-1.5708 0 0"/>
 </robot>
